File: bmek-master/pcb/v3/BMEK_Solder/noname.kicad_pcb (KiCad board)
At the start: 2 copper layers, 353.8 x 116.1 mm, 0 parts

Commit message: update 17:18 28/01/2021
Parts:
- added U1: E73-2G4M04S-52832, fruitkt:E73-2G4M08S1C, B.Cu at (50.7, 51.9)
Other:
- net class Default added: clearance 0.2, trace_width 0.25, via_dia 0.8, via_drill 0.4
