File: arisu-pcb/arisu.kicad_pcb (KiCad board)
At the start: 2 copper layers, 339.1 x 118.7 mm, 176 parts, among them J1 USB_B_Micro, SW1 SW_Push, SW10 SW_Push, SW11 SW_Push, SW12 SW_Push, SW13 SW_Push, SW14 SW_Push, SW15 SW_Push, SW16 SW_Push, SW17 SW_Push, SW18 SW_Push, SW19 SW_Push, SW2 SW_Push, SW20 SW_Push, SW21 SW_Push, SW22 SW_Push, SW23 SW_Push, SW24 SW_Push, SW25 SW_Push, SW26 SW_Push, SW27 SW_Push, SW28 SW_Push, SW29 SW_Push, SW3 SW_Push, SW30 SW_Push, SW31 SW_Push, SW32 SW_Push, SW33 SW_Push, SW34 SW_Push, SW35 SW_Push, SW36 SW_Push, SW37 SW_Push, SW38 SW_Push, SW39 SW_Push, SW4 SW_Push, SW40 SW_Push, SW41 SW_Push, SW42 SW_Push, SW43 SW_Push, SW44 SW_Push, SW45 SW_Push, SW46 SW_Push, SW47 SW_Push, SW48 SW_Push, SW49 SW_Push, SW5 SW_Push, SW50 SW_Push, SW51 SW_Push, SW52 SW_Push, SW53 SW_Push, SW54 SW_Push, SW55 SW_Push, SW56 SW_Push, SW57 SW_Push, SW58 SW_Push, SW59 SW_Push, SW6 SW_Push, SW60 SW_Push, SW61 SW_Push, SW62 SW_Push, SW63 SW_Push, SW64 SW_Push, SW65 SW_Push, SW66 SW_Push, SW67 SW_Push, SW7 SW_Push, SW8 SW_Push, SW9 SW_Push, U1 USBLC6-2SC6, U2 ATmega32U4-AU, Y1 Crystal_GND24

Commit message: add some keyboard
Parts:
- removed G*** (x2): LOGO, arisu:arisu-logo
- removed U2: ATmega32U4-AU, Housings_QFP:TQFP-44_10x10mm_Pitch0.8mm
- added U3: AT90USB1286-MU, Package_DFN_QFN:QFN-64-1EP_9x9mm_P0.5mm_EP7.5x7.5mm, B.Cu at (175.5, 42.2)
- D1, D10, D11, D12, D13, D14, D15, D16, D17, D18, D19, D2, D20, D21, D22, D23, D24, D25, D26, D27, D28, D29, D3, D30, D31, D32, D33, D34, D35, D36, D37, D38, D39, D4, D40, D41, D42, D43, D44, D45, D46, D47, D48, D49, D5, D50, D51, D52, D53, D54, D55, D56, D57, D58, D59, D6, D60, D61, D62, D63, D64, D65, D66, D67, D7, D8, D9: footprint Diodes_SMD:D_SOD-123 -> Diode_SMD:D_SOD-123
- renumbered PF6 to J10, PF7 to J11, VCC to J12, D+ to J13, D- to J14, GND to J15, MISO to J2, VCC to J3, SCK to J4, MOSI to J5, RES to J6, GND to J7, PF4 to J8, PF5 to J9
Routing:
- net /row4: track 433.8 -> 377.4 mm
- net Net-(U3-Pad22): track 0.00 -> 1.95 mm, vias 0 -> 1
- net GND: track 71.6 -> 69.6 mm, vias 12 -> 11
- removed copper zone on F.Cu, net GND

Commit message: cap nhat 18:16 27/2/2021
Parts:
- removed U3: AT90USB1286-MU, Package_DFN_QFN:QFN-64-1EP_9x9mm_P0.5mm_EP7.5x7.5mm
- added G***: LOGO, arisu:arisu-logo, B.Cu at (287.0, 114.9)
- added G***: LOGO, arisu:arisu-logo, F.Cu at (287.0, 117.3)
- added U2: ATmega32U4-AU, Housings_QFP:TQFP-44_10x10mm_Pitch0.8mm, B.Cu at (175.5, 42.2)
- D1, D10, D11, D12, D13, D14, D15, D16, D17, D18, D19, D2, D20, D21, D22, D23, D24, D25, D26, D27, D28, D29, D3, D30, D31, D32, D33, D34, D35, D36, D37, D38, D39, D4, D40, D41, D42, D43, D44, D45, D46, D47, D48, D49, D5, D50, D51, D52, D53, D54, D55, D56, D57, D58, D59, D6, D60, D61, D62, D63, D64, D65, D66, D67, D7, D8, D9: footprint Diode_SMD:D_SOD-123 -> Diodes_SMD:D_SOD-123
- renumbered J13 to D+, J14 to D-, J7 to GND, J15 to GND, J2 to MISO, J5 to MOSI, J8 to PF4, J9 to PF5, J10 to PF6, J11 to PF7, J6 to RES, J4 to SCK, J3 to VCC, J12 to VCC
Routing:
- net /row4: track 377.4 -> 433.8 mm
- net Net-(U3-Pad22): track 1.95 -> 0.00 mm, vias 1 -> 0
- net GND: track 69.6 -> 71.6 mm, vias 11 -> 12
- added copper zone on F.Cu, net GND
