File: anavi-macro-pad-8/anavi-macro-pad-8.sch (KiCad schematic (older format))
At the start: 45 parts, among them J1 USB_B_Micro, J2 Conn_01x04_Female, J3 Conn_01x03_Male, J4 Conn_01x03_Male, J5 AVR-ISP-6, Q1 Q_NPN_BEC, SW1 SW_DIP_x01, SW2 SW_DIP_x01, SW3 SW_DIP_x01, SW4 SW_DIP_x01, SW5 SW_DIP_x01, SW6 SW_DIP_x01, SW7 SW_DIP_x01, SW8 SW_DIP_x01, SW9 SW_DIP_x01, U1 ATmega32U4-AU, Y1 Crystal

Commit message: cap nhat 18:16 27/2/2021
Parts:
- J1: symbol Connector:USB_B_Micro -> anavi-macro-pad-8-rescue:USB_B_Micro-Connector
Changed lines of the file:
@@
 $EndDescr
 $Comp
-L Connector:USB_B_Micro J1
+L anavi-macro-pad-8-rescue:USB_B_Micro-Connector J1
 U 1 1 5EACE252
 P 950 3300
