File: tool/nrfmicro/hardware/nrfmicro.sch (KiCad schematic (older format))
At the start: 25 parts, among them J1 USB-C Conn, J2 SWD, J3 Ex_Bat, J4 Ex_USB, J5 , J6 , Q1 AO3407, Q2 AO3407, U1 E73-2G4M08S1C, U2 XC6220B331MR-G, U3 TP4054, U4 ProMicro, X1 32.768kHz

Commit message: update 17:18 28/01/2021
Parts:
- removed J4: Ex_USB, nrfmicro:connector_usb, symbol Connector_Generic:Conn_01x04

Commit message: cap nhat 18:16 27/2/2021
Parts:
- added J4: Data +, Connector_PinSocket_2.54mm:PinSocket_1x01_P2.54mm_Vertical, symbol Connector_Generic:Conn_01x01
- added J7: Data -, Connector_PinSocket_2.54mm:PinSocket_1x01_P2.54mm_Vertical, symbol Connector_Generic:Conn_01x01
Connections:
- net DATA+: now also J4.1 (Pin_1)
- net DATA-: now also J7.1 (Pin_1)
Changed lines of the file:
@@
 	1    0    0    -1
 $EndComp
+$Comp
+L Connector_Generic:Conn_01x01 J4
+U 1 1 602E939F
+P 8100 2075
+F 0 "J4" V 8064 1987 50  0000 R CNN
+F 1 "Data +" V 7973 1987 50  0000 R CNN
+F 2 "Connector_PinSocket_2.54mm:PinSocket_1x01_P2.54mm_Vertical" H 8100 2075 50  0001 C CNN
+F 3 "~" H 8100 2075 50  0001 C CNN
+	1    8100 2075
+	0    -1   -1   0
+$EndComp
+$Comp
+L Connector_Generic:Conn_01x01 J7
+U 1 1 602EA25D
+P 8575 2075
+F 0 "J7" V 8539 1987 50  0000 R CNN
+F 1 "Data -" V 8448 1987 50  0000 R CNN
+F 2 "Connector_PinSocket_2.54mm:PinSocket_1x01_P2.54mm_Vertical" H 8575 2075 50  0001 C CNN
+F 3 "~" H 8575 2075 50  0001 C CNN
+	1    8575 2075
+	0    -1   -1   0
+$EndComp
+Text GLabel 8575 2275 3    60   Input ~ 0
+DATA-
+Text GLabel 8100 2275 3    60   Input ~ 0
+DATA+
 $EndSCHEMATC
