File: Hub20/hardware/1.0/Hub20.kicad_pcb (KiCad board)
At the start: 2 copper layers, 89 x 124 mm, 183 parts, among them J1 USB_C_Receptacle_USB2.0, J2 USB_C_Receptacle_USB2.0, J3 USB_C_Receptacle_USB2.0, J4 USB_C_Receptacle_USB2.0, Q1 DTC123J, Q2 BSS138, SW1 EVQPUL, SW10 MX_RGB, SW11 MX_RGB, SW12 MX_RGB, SW13 EC11, SW14 MX_RGB, SW15 MX_RGB, SW16 MX_RGB, SW17 MX_RGB, SW18 MX_RGB, SW19 MX_RGB, SW2 MX_RGB, SW20 MX_RGB, SW21 MX_RGB, SW22 MX_RGB, SW23 MX_RGB, SW3 MX_RGB, SW4 MX_RGB, SW5 MX_RGB, SW6 MX_RGB, SW7 EC11, SW8 MX_RGB, SW9 MX_RGB, U1 AP2112K-3.3, U2 USBLC6-2SC6, U3 STM32F072C8Tx, U5 CY7C65632-28LTXCT, U6 USBLC6-2SC6, U7 USBLC6-2SC6, U8 USBLC6-2SC6, Y1 12MHz

Commit message: update 22:15 31/01/2021
Routing:
- net +3.3VA: track 48.5 -> 47.1 mm

Commit message: cap nhat 12:00 18/03/2021
Routing:
- net /R5: track 111.2 -> 107.1 mm
