File: comet46-nnyc/comet46-nnyc.kicad_pcb (KiCad board)
At the start: 2 copper layers, 134.6 x 97 mm, 26 parts, among them SW1 , SW10 , SW11 , SW12 , SW13 , SW14 , SW15 , SW16 , SW17 , SW18 , SW19 , SW2 , SW20 , SW21 , SW22 , SW23 , SW3 , SW4 , SW5 , SW6 , SW7 , SW8 , SW9 , U1 MDBT40-256RV3, U2 MDBT40-256RV3, Y1 Crystal_Small

Commit message: cap nhat 18:16 27/2/2021
Parts:
- turned SW21 to 355 degrees
- turned SW22 to 347.5 degrees
Other:
- outline, holes or cut-outs redrawn

Commit message: cap nhat 12:00 18/03/2021
Parts:
- removed U2: MDBT40-256RV3, fruitkt:MDBT40-256RV3
- removed Y1: Crystal_Small, Crystal:Crystal_SMD_3215-2Pin_3.2x1.5mm
- added BT1: , Battery:BatteryHolder_Keystone_1060_1x2032, F.Cu at (73.5, 113.8)
- added BT2: , Battery:BatteryHolder_Keystone_1060_1x2032, B.Cu at (73.5, 113.8)
- added C1: C, Capacitor_SMD:C_0603_1608Metric_Pad1.08x0.95mm_HandSolder, F.Cu at (104.9, 121.9)
- added C2: C, Capacitor_SMD:C_0603_1608Metric_Pad1.08x0.95mm_HandSolder, B.Cu at (97.0, 121.9)
- added J1: , Connector_PinHeader_2.54mm:PinHeader_1x04_P2.54mm_Horizontal, F.Cu at (93.5, 125.0)
- added Q1: SI2302, Package_TO_SOT_SMD:SOT-23_Handsoldering, F.Cu at (101.0, 121.9)
- added Q2: SI2302, Package_TO_SOT_SMD:SOT-23_Handsoldering, B.Cu at (101.0, 121.9)
- added SW24: , Button_Switch_SMD:SW_SPDT_PCM12, F.Cu at (101.5, 128.3)
- added SW25: , Button_Switch_SMD:SW_SPDT_PCM12, B.Cu at (101.5, 128.3)
- added U3: Core51822B-Left, fruitkt:Core51822B, B.Cu at (115.6, 118.1)
- U1: value MDBT40-256RV3 -> Core51822B-Right; footprint fruitkt:MDBT40-256RV3 -> fruitkt:Core51822B
- moved U1 0.69 mm to (115.6, 118.1), turned to 180 degrees
- turned SW20 to 348 degrees
- renumbered SW4 to SW10, SW18 to SW12, SW5 to SW13, SW12 to SW14, SW19 to SW15, SW21 to SW16, SW6 to SW17, SW13 to SW18, SW20 to SW19, SW8 to SW2, SW22 to SW20, SW7 to SW21, SW14 to SW22, SW15 to SW3, SW2 to SW4, SW9 to SW5, SW16 to SW6, SW3 to SW7, SW10 to SW8, SW17 to SW9
Connections:
- SW1 pad 1: Net-(SW1-Pad1) -> SW1
- SW10 pad 1: Net-(SW4-Pad1) -> SW10
- SW11 pad 1: Net-(SW11-Pad1) -> SW11
- SW12 pad 1: Net-(SW18-Pad1) -> SW12
- SW13 pad 1: Net-(SW5-Pad1) -> SW13
- SW14 pad 1: Net-(SW12-Pad1) -> SW14
- SW15 pad 1: Net-(SW19-Pad1) -> SW15
- SW16 pad 1: Net-(SW21-Pad1) -> SW16
- SW17 pad 1: Net-(SW6-Pad1) -> SW17
- SW18 pad 1: Net-(SW13-Pad1) -> SW18
- SW19 pad 1: Net-(SW20-Pad1) -> SW19
- SW2 pad 1: Net-(SW8-Pad1) -> SW2
- SW20 pad 1: Net-(SW22-Pad1) -> SW20
- SW21 pad 1: Net-(SW7-Pad1) -> SW21
- SW22 pad 1: Net-(SW14-Pad1) -> SW22
- SW23 pad 1: Net-(SW23-Pad1) -> SW23
- SW3 pad 1: Net-(SW15-Pad1) -> SW3
- SW4 pad 1: Net-(SW2-Pad1) -> SW4
- SW5 pad 1: Net-(SW9-Pad1) -> SW5
- SW6 pad 1: Net-(SW16-Pad1) -> SW6
- SW7 pad 1: Net-(SW3-Pad1) -> SW7
- SW8 pad 1: Net-(SW10-Pad1) -> SW8
- SW9 pad 1: Net-(SW17-Pad1) -> SW9
- U1 pad 1: Net-(U1-Pad1) -> GND
- U1 pad 11: Net-(U1-Pad11) -> GND
- U1 pad 12: Net-(U1-Pad12) -> VCC
- U1 pad 13: Net-(U1-Pad1) -> SW3
- U1 pad 14: Net-(U1-Pad14) -> SW2
- U1 pad 15: Net-(U1-Pad15) -> SW1
- U1 pad 16: Net-(U1-Pad16) -> SW4
- U1 pad 17: Net-(U1-Pad17) -> SW6
- U1 pad 18: Net-(U1-Pad18) -> SW5
- U1 pad 19: Net-(U1-Pad19) -> SW7
- U1 pad 2: Net-(U1-Pad1) -> SW21
- U1 pad 22: Net-(U1-Pad22) -> SW8
- U1 pad 23: Net-(U1-Pad23) -> SW9
- U1 pad 25: Net-(U1-Pad1) -> Net-(U1-Pad25)
- U1 pad 26: Net-(U1-Pad26) -> SW10
- U1 pad 27: Net-(U1-Pad27) -> SW11
- U1 pad 28: Net-(U1-Pad28) -> SW12
- U1 pad 29: Net-(U1-Pad29) -> SW13
- U1 pad 3: Net-(U1-Pad3) -> SW22
- U1 pad 30: Net-(U1-Pad30) -> SW14
- U1 pad 31: Net-(U1-Pad31) -> SWDIO
- U1 pad 32: Net-(U1-Pad32) -> SWCLK
- U1 pad 33: Net-(U1-Pad33) -> SW15
- U1 pad 34: Net-(U1-Pad34) -> SW17
- U1 pad 35: Net-(U1-Pad35) -> SW18
- U1 pad 36: Net-(U1-Pad36) -> SW19
- U1 pad 4: Net-(U1-Pad4) -> SW23
- U1 pad 5: Net-(U1-Pad5) -> SW20
- U1 pad 6: Net-(U1-Pad6) -> SW16
Routing:
- net (no net): track 372.7 -> 0.00 mm, vias 27 -> 0
- net SW13: track 0.00 -> 179.1 mm, vias 0 -> 1
- net SW22: track 0.00 -> 179.0 mm, vias 0 -> 1
- net GND: track 3.48 -> 165.9 mm, vias 2 -> 3
- net SW11: track 0.00 -> 155.0 mm, vias 0 -> 1
- net Net-(U1-Pad1): track 133.4 -> 0.00 mm, vias 9 -> 0
- net SW1: track 0.00 -> 117.4 mm, vias 0 -> 1
- net SW17: track 0.00 -> 113.3 mm, vias 0 -> 1
- net SW21: track 0.00 -> 108.8 mm, vias 0 -> 2
- net SW10: track 0.00 -> 99.9 mm, vias 0 -> 3
- net SW18: track 0.00 -> 95.8 mm, vias 0 -> 1
- net SW4: track 0.00 -> 85.2 mm, vias 0 -> 2
- net SW19: track 0.00 -> 79.9 mm, vias 0 -> 1
- net SW14: track 0.00 -> 79.1 mm, vias 0 -> 1
- net SW23: track 0.00 -> 75.6 mm, vias 0 -> 1
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- added copper zone on B.Cu, net (none)
- added copper zone on F.Cu, net (none)
- added copper zone on B.Cu, net GND
- added copper zone on F.Cu, net GND
Other:
- net class Default: clearance 0.2 -> 0.4; trace_width 0.25 -> 0.4
- rule trace_clearance: 0.2 -> 0.4
- board text added: "3.3v"
- board text added: "DIO"
- board text added: "GND"
- board text added: "LEFT"
- board text added: "RIGHT"
- board text added: "SCK"
- board text added: "y=97,0026 x=134,62"
