File: comet46-nnyc/comet46-nnyc.sch (KiCad schematic (older format))
At the start: 26 parts, among them SW1 , SW10 , SW11 , SW12 , SW13 , SW14 , SW15 , SW16 , SW17 , SW18 , SW19 , SW2 , SW20 , SW21 , SW22 , SW23 , SW3 , SW4 , SW5 , SW6 , SW7 , SW8 , SW9 , U1 MDBT40-256RV3, U2 MDBT40-256RV3, Y1 Crystal_Small

Commit message: cap nhat 12:00 18/03/2021
Parts:
- removed U1, U2: MDBT40-256RV3, fruitkt:MDBT40-256RV3, symbol fruitkt:MDBT40-256RV3
- removed Y1: Crystal_Small, Crystal:Crystal_SMD_3215-2Pin_3.2x1.5mm, symbol Device:Crystal_Small
- added BT1, BT2: (no value), Battery:BatteryHolder_Keystone_1060_1x2032, symbol Device:Battery_Cell
- added C1, C2: C, Capacitor_SMD:C_0603_1608Metric_Pad1.08x0.95mm_HandSolder, symbol Device:C
- added J1: (no value), Connector_PinHeader_2.54mm:PinHeader_1x04_P2.54mm_Horizontal, symbol Connector_Generic:Conn_01x04
- added Q1, Q2: SI2302, Package_TO_SOT_SMD:SOT-23_Handsoldering, symbol SI2302:SI2302
- added SW24, SW25: (no value), Button_Switch_SMD:SW_SPDT_PCM12, symbol Switch:SW_DPDT_x2
- added U1: Core51822B-Right, fruitkt:Core51822B, symbol fruitkt:Core51822B
- added U3: Core51822B-Left, fruitkt:Core51822B, symbol fruitkt:Core51822B
- renumbered SW4 to SW10, SW18 to SW12, SW5 to SW13, SW12 to SW14, SW19 to SW15, SW21 to SW16, SW6 to SW17, SW13 to SW18, SW20 to SW19, SW8 to SW2, SW22 to SW20, SW7 to SW21, SW14 to SW22, SW15 to SW3, SW2 to SW4, SW9 to SW5, SW16 to SW6, SW3 to SW7, SW10 to SW8, SW17 to SW9
Connections:
- net labels added: SW1, SW10, SW11, SW12, SW13, SW14, SW15, SW16, SW17, SW18, SW19, SW2, SW20, SW21, SW22, SW23, SW3, SW4, SW5, SW6, SW7, SW8, SW9, SWCLK, SWDIO, VCC
- wire segments 0 -> 22
Other:
- moved on the sheet: SW1, SW10, SW11, SW12, SW13, SW14, SW15, SW16, SW17, SW18, SW19, SW2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
