File: redox-w/pcb/redox_w_transmitters_kicad_files/redox_rev1.sch (KiCad schematic (older format))
At the start: 83 parts, among them K0 KEYSW, K1 KEYSW, K10 KEYSW, K11 KEYSW, K12 KEYSW, K13 KEYSW, K14 KEYSW, K15 KEYSW, K16 KEYSW, K2 KEYSW, K20 KEYSW, K21 KEYSW, K22 KEYSW, K23 KEYSW, K24 KEYSW, K25 KEYSW, K26 KEYSW, K3 KEYSW, K30 KEYSW, K31 KEYSW, K32 KEYSW, K33 KEYSW, K34 KEYSW, K35 KEYSW, K36 KEYSW, K4 KEYSW, K40 KEYSW, K41 KEYSW, K42 KEYSW, K43 KEYSW, K44 KEYSW, K45 KEYSW, K46 KEYSW, K5 KEYSW, K6 KEYSW

Commit message: cap nhat 12:00 18/03/2021
Parts:
- removed H1, H2, H3, H4, H5, H6: (no value), fruitkey:Hole_M3, symbol Mechanical:MountingHole
- BT_LEFT1, BT_RIGHT1: footprint Battery:BatteryHolder_Keystone_3034_1x20mm -> redox_w_footprints:BatteryHolder_Keystone_3034_1x20mm
- D0, D1, D10, D11, D12, D13, D14, D15, D16, D2, D20, D21, D22, D23, D24, D25, D26, D3, D30, D31, D32, D33, D34, D35, D36, D4, D40, D41, D42, D43, D44, D45, D46, D5, D6: footprint fruitkey:Diode_smd -> redox_w_footprints:Diode-dual
- J_PROG_PORT1: footprint Connector_PinHeader_2.54mm:PinHeader_1x04_P2.54mm_Horizontal -> Connector_PinHeader_2.54mm:PinHeader_1x04_P2.54mm_Vertical
- K0, K1, K10, K11, K12, K13, K14, K15, K16, K2, K20, K21, K22, K23, K24, K25, K26, K3, K30, K31, K32, K33, K34, K35, K36, K4, K40, K41, K42, K43, K44, K45, K46, K5, K6: footprint Switch_2_mat:1u -> redox_w_footprints:Mx_Alps_100-dualside
